Commit message: Código completado

File: description/robot.urdf.xacro (robot description, xacro)
@@ -2,4 +2,5 @@
 <robot xmlns:xacro="http://www.ros.org/wiki/xacro"  name="robot">
     <!-- Ejemplo de comentario -->
+    <xacro:include filename = "inertial_macros.xacro"/>
     <xacro:include filename = "robot_core.xacro"/>
 </robot>

File: description/robot_core.xacro (robot description, xacro)
@@ -14,5 +14,6 @@
         <color rgba = "0 0 0 1"/>
     </material>
-    <!-- Defino la geometría del modelo físico -->
+    <!-- Geometría del modelo físico -->
+    <!-- base_link-->
     <link name = "base_link">
     </link>
@@ -22,4 +23,5 @@
         <origin xyz = "-0.1 0 0"/>
     </joint>
+    <!-- Chassis link -->
     <link name = "chassis">
         <visual>
@@ -30,4 +32,81 @@
             <material name = "white"/>
         </visual>
+        <collision>
+            <origin xyz = "0.15 0 0.075"/>
+            <geometry>
+                <box size = "0.3 0.3 0.15"/>    <!-- Defino el tamaño (en m) de la "caja" que será mi robot -->
+            </geometry>
+        </collision>
+        <xacro:inertial_box mass="0.5" x="0.3" y="0.3" z="0.15">
+            <origin xyz="0.15 0 0.075" rpy="0 0 0"/>
+        </xacro:inertial_box>
+    </link>
+    <!-- Rueda izquierda link -->
+    <joint name = "left_wheel_joint" type = "continuous">
+        <parent link = "base_link"/>
+        <child link = "left_wheel"/>
+        <origin xyz = "0 0.175 0" rpy = "-${pi/2} 0 0"/>
+        <axis xyz = "0 0 1"/>
+    </joint>
+    <link name = "left_wheel">
+        <visual>
+            <geometry>
+                <cylinder radius = "0.05" length = "0.04"/>
+            </geometry>
+            <material name = "blue"/>
+        </visual>
+        <collision>
+            <geometry>
+                <cylinder radius = "0.05" length = "0.04"/>
+            </geometry>
+        </collision>
+        <xacro:inertial_cylinder mass="0.1" length="0.05" radius="0.05">
+            <origin xyz="0 0 0" rpy="0 0 0"/>
+        </xacro:inertial_cylinder>
+    </link>
+    <!-- Rueda derecha link -->
+    <joint name = "right_wheel_joint" type = "continuous">
+        <parent link = "base_link"/>
+        <child link = "right_wheel"/>
+        <origin xyz = "0 -0.175 0" rpy = "${pi/2} 0 0"/>
+        <axis xyz = "0 0 -1"/>
+    </joint>
+    <link name = "right_wheel">
+        <visual>
+            <geometry>
+                <cylinder radius = "0.05" length = "0.04"/>
+            </geometry>
+            <material name = "blue"/>
+        </visual>
+        <collision>
+            <geometry>
+                <cylinder radius = "0.05" length = "0.04"/>
+            </geometry>
+        </collision>
+        <xacro:inertial_cylinder mass="0.1" length="0.05" radius="0.05">
+            <origin xyz="0 0 0" rpy="0 0 0"/>
+        </xacro:inertial_cylinder>
+    </link>
+    <!-- Rueda loca (caster wheel) link -->
+    <joint name = "caster_wheel_joint" type = "fixed">
+        <parent link = "chassis"/>
+        <child link = "caster_wheel"/>
+        <origin xyz = "0.24 0 0"/>
+    </joint>
+    <link name = "caster_wheel">
+        <visual>
+            <geometry>
+                <sphere radius = "0.05"/>
+            </geometry>
+            <material name = "black"/>
+        </visual>
+        <collision>
+            <geometry>
+                <sphere radius = "0.05"/>
+            </geometry>
+        </collision>
+        <xacro:inertial_sphere mass="0.1" radius="0.05">
+            <origin xyz="0 0 0" rpy="0 0 0"/>
+        </xacro:inertial_sphere>
     </link>
 </robot>
